File: hardware/STM32_hardware/STM32_hardware.kicad_pcb (KiCad board)
At the start: 2 copper layers, 23 parts, among them J1 Conn_02x07_Odd_Even, J2 Power, J3 Output, J4 Input, U1 STM32L021K4Tx, U2 MCP4801, U3 BU33SD5WG-TR

Commit message: harware_PCB_contour
Parts:
- added H1: MountingHole_Pad, MountingHole:MountingHole_3.2mm_M3_Pad, F.Cu at (99.1, 44.4)
- added H2: MountingHole_Pad, MountingHole:MountingHole_3.2mm_M3_Pad, F.Cu at (149.1, 44.4)
- added H3: MountingHole_Pad, MountingHole:MountingHole_3.2mm_M3_Pad, F.Cu at (99.1, 84.4)
- added H4: MountingHole_Pad, MountingHole:MountingHole_3.2mm_M3_Pad, F.Cu at (149.1, 84.4)
- moved J3 38.6 mm to (149.1, 64.4), turned to -90 degrees
- moved J2 19.3 mm to (124.1, 44.4)
- moved J4 14.8 mm to (99.1, 64.4), turned to 90 degrees
Other:
- board outline added: 58.7 x 48.7 mm

Commit message: Hardware_routin
Parts:
- C1: value 100nF -> 4.7uF
- moved U3 42.5 mm to (136.1, 47.1), turned to -90 degrees
- moved D1 38.7 mm to (105.7, 45.7), turned to 180 degrees
- moved D3 37.7 mm to (109.6, 45.7), turned to 180 degrees
- moved R4 35.0 mm to (109.6, 49.0), turned to 180 degrees
- moved R1 33.3 mm to (105.5, 49.0), turned to 180 degrees
- moved C8 23.5 mm to (141.5, 47.0), turned to 90 degrees
- moved R2 19.8 mm to (122.4, 56.1), turned to 90 degrees
- moved C1 19.6 mm to (132.6, 70.4), turned to -90 degrees
- moved L1 16.6 mm to (113.0, 61.2), turned to -90 degrees
- moved C7 15.1 mm to (132.5, 47.0), turned to -90 degrees
- moved C10 14.0 mm to (123.2, 82.3), turned to 180 degrees
- moved C9 13.7 mm to (123.2, 79.0), turned to 180 degrees
- moved C3 12.9 mm to (129.0, 70.4), turned to -90 degrees
- moved U2 11.8 mm to (123.2, 74.2), turned to 180 degrees
- moved U1 11.3 mm to (124.1, 64.4)
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Connections:
- C1 pad 1: +3V3 -> +3.3V
- C2 pad 1: +3V3 -> +3.3V
- C3 pad 1: +3V3 -> +3.3V
- C8 pad 1: +3V3 -> +3.3V
- D3 pad 2: +3V3 -> +3.3V
- L1 pad 1: +3V3 -> +3.3V
- U3 pad 5: +3V3 -> +3.3V
Routing:
- net +3.3V: track 0.00 -> 91.1 mm
- net +3.3VA: track 0.00 -> 41.5 mm, vias 0 -> 2
- net LED_STATUS: track 0.00 -> 39.5 mm, vias 0 -> 2
- net DAC_OUT: track 0.00 -> 39.0 mm, vias 0 -> 2
- net NRST: track 0.00 -> 30.4 mm, vias 0 -> 2
- net USART2_TX: track 0.00 -> 26.4 mm, vias 0 -> 2
- net GND: track 0.00 -> 24.4 mm, vias 0 -> 2
- net ADC_IN1: track 0.00 -> 24.3 mm
- net SWDIO: track 0.00 -> 23.2 mm, vias 0 -> 2
- net +5V: track 0.00 -> 21.3 mm, vias 0 -> 2
- net Net-(U3-GND): track 0.00 -> 21.0 mm, vias 0 -> 2
- net SWDCLK: track 0.00 -> 17.7 mm, vias 0 -> 2
- net USART2_RX: track 0.00 -> 16.5 mm, vias 0 -> 2
- net DAC_nCS: track 0.00 -> 8.11 mm
- net SPI1_SCK: track 0.00 -> 6.51 mm
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- added copper zone on B.Cu, net GND
- added copper zone on F.Cu, net GND
Other:
- board size 58.7 x 48.7 mm -> 59 x 49 mm
- rule pad_to_mask_clearance: 0 -> 0.1
