File: hardware/STM32_hardware/STM32_hardware.kicad_pcb (KiCad board)
At the start: 2 copper layers, 59 x 49 mm, 27 parts, among them J1 Conn_02x07_Odd_Even, J2 Power, J3 Output, J4 Input, U1 STM32L021K4Tx, U2 MCP4801, U3 BU33SD5WG-TR

Commit message: Hardware_routing
Other:
- board text added: "Amine KACHKACH Etienne PARMENTIER"
Changed lines of the file:
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@@
   (gr_arc (start 94.676696 44.684265) (mid 95.876072 41.423709) (end 99.060031 40.033697)
     (stroke (width 0.1) (type default)) (layer "Edge.Cuts"))
+  (gr_text "Amine KACHKACH\nEtienne PARMENTIER" (at 104.14 81.28) (layer "F.Cu")
+    (effects (font (size 1 1) (thickness 0.25) bold) (justify left bottom))
+  )
   (segment (start 122 42.2) (end 121.25 42.95) (width 0.6) (layer "F.Cu") (net 1))
   (segment (start 108.599 49.022) (end 108.599 49.024082) (width 0.6) (layer "F.Cu") (net 1))

Commit message: Hardware_routing_emoji
Other:
- board text added: "Amine KACHKACH :) Etienne PARMENTIER :)"
- board text removed: "Amine KACHKACH Etienne PARMENTIER"
Changed lines of the file:
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@@
   (gr_arc (start 94.676696 44.684265) (mid 95.876072 41.423709) (end 99.060031 40.033697)
     (stroke (width 0.1) (type default)) (layer "Edge.Cuts"))
-  (gr_text "Amine KACHKACH\nEtienne PARMENTIER" (at 104.14 81.28) (layer "F.Cu")
+  (gr_text "Amine KACHKACH		:)\nEtienne PARMENTIER	:)\n" (at 102.235 81.915) (layer "F.Cu")
     (effects (font (size 1 1) (thickness 0.25) bold) (justify left bottom))
   )
