File: hardware/STM32_hardware/STM32_hardware.kicad_sch (KiCad schematic)
At the start: 11 parts, among them U1 STM32L021K4Tx

Commit message: schema de principe
Parts:
- added C10: 10uF, Capacitor_SMD:C_0805_2012Metric_Pad1.18x1.45mm_HandSolder, symbol Device:C_Small
- added C7, C8: 1uF, Capacitor_SMD:C_0805_2012Metric_Pad1.18x1.45mm_HandSolder, symbol Device:C_Small
- added C9: 100nF, Capacitor_SMD:C_0805_2012Metric_Pad1.18x1.45mm_HandSolder, symbol Device:C_Small
- added D3: Green LED, LED_SMD:LED_0603_1608Metric_Pad1.05x0.95mm_HandSolder, symbol Device:LED_Small
- added J1: Conn_02x07_Odd_Even, Connector_PinHeader_1.27mm:PinHeader_2x07_P1.27mm_Vertical_SMD, symbol Connector_Generic:Conn_02x07_Odd_Even
- added J2: Power, Connector_JST:JST_XH_B2B-XH-A_1x02_P2.50mm_Vertical, symbol Connector_Generic:Conn_01x02
- added J3: Output, Connector_JST:JST_XH_B2B-XH-A_1x02_P2.50mm_Vertical, symbol Connector_Generic:Conn_01x02
- added J4: Input, Connector_JST:JST_XH_B2B-XH-A_1x02_P2.50mm_Vertical, symbol Connector_Generic:Conn_01x02
- added R4: 1K, Resistor_SMD:R_0805_2012Metric_Pad1.20x1.40mm_HandSolder, symbol Device:R_Small
- added U2: MCP4801, Package_SO:SOIC-8_3.9x4.9mm_P1.27mm, symbol Analog_DAC:MCP4801
- added U3: BU33SD5WG-TR, Package_TO_SOT_SMD:SOT-23-5, symbol Regulator_Linear:MCP1802x-xx02xOT
- C1, C2, C3, C4, C5, C6: footprint (none) -> Capacitor_SMD:C_0805_2012Metric_Pad1.18x1.45mm_HandSolder
- D1: footprint (none) -> LED_SMD:LED_0603_1608Metric_Pad1.05x0.95mm_HandSolder
- L1: footprint (none) -> Inductor_SMD:L_0805_2012Metric_Pad1.05x1.20mm_HandSolder
- R1, R2: footprint (none) -> Resistor_SMD:R_0805_2012Metric_Pad1.20x1.40mm_HandSolder
Connections:
- net +3.3V: now also J1.3 (Pin_3)
- net +3.3VA: now also C10.1, C9.1, U2.1 (Vdd), U2.6 (~{SHDN})
- net +3V3: now also C8.1, D3.2 (A), U3.5 (VOUT)
- net ADC_IN1: now also J4.1 (Pin_1)
- net DAC_nCS: now also U2.2 (~{CS})
- net DAC_nLDAC: now also U2.5 (~{LDAC})
- net GND: now also C10.2, C9.2, J1.11 (Pin_11), J1.5 (Pin_5), J1.7 (Pin_7), J2.2 (Pin_2), J3.2 (Pin_2), J4.2 (Pin_2), R4.2, U2.7 (Vss)
- net NRST: now also J1.12 (Pin_12)
- net SPI1_MOSI: now also U2.4 (SDI)
- net SPI1_SCK: now also U2.3 (SCK)
- net SWDCLK: now also J1.6 (Pin_6)
- net SWDIO: now also J1.4 (Pin_4)
- net USART2_RX: now also J1.13 (Pin_13)
- net USART2_TX: now also J1.14 (Pin_14)
- new net: C7.2, C8.2, U3.2 (GND)
- new net: D3.1 (K), R4.1
- new net +5V: C7.1, J2.1 (Pin_1), U3.1 (VIN), U3.3 (~{SHDN})
- new net DAC_OUT: J3.1 (Pin_1), U2.8 (Vout)
- no-connect marks 16 -> 20
Other:
- moved on the sheet: C1, C2, C3, C4, C5, L1

Commit message: harware_PCB_contour
Parts:
- added H1, H2, H3, H4: MountingHole_Pad, MountingHole:MountingHole_3.2mm_M3_Pad, symbol Mechanical:MountingHole_Pad
Connections:
- net GND: now also H1.1, H2.1, H3.1, H4.1
Other:
- moved on the sheet: C1, C10, C2, C3, C4, C5, C6, C7, C8, C9, D3, L1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

Commit message: Hardware_routin
Parts:
- C1: value 100nF -> 4.7uF
Connections:
- net +3V3 is gone; now on net +3.3V: C1.1, C2.1, C3.1, C8.1, D3.2 (A), L1.1, U3.5 (VOUT)
